Commit message: Final before put on Raspberry Pi 4B

File: src/cnc_description/urdf/cnc.urdf (robot description, URDF)
Before this commit: robot cncweld, 5 links, 4 joints
Joints:
- joint Z_axis_tool0_joint: origin xyz=0.0 0.0 0.0 rpy=0.0 0.0 0.0 -> xyz=0.045 0.0 0.0 rpy=0.0 0.0 0.0

Commit message: urdf completed

File: src/cnc_description/urdf/cnc.urdf (robot description, URDF)
Before this commit: robot cncweld, 5 links, 4 joints
Joints:
- joint X_axis_Y_axis_joint: limit lower=0.0 upper=1.0 effort=1000.0 velocity=0.05 -> lower=0.0 upper=0.7 effort=1000.0 velocity=0.05
- joint Z_axis_tool0_joint: limit lower=0.0 upper=0.2 effort=1000.0 velocity=0.05 -> lower=0.0 upper=0.086 effort=1000.0 velocity=0.05; origin xyz=0.045 0.0 0.0 rpy=0.0 0.0 0.0 -> xyz=0.31 0.046 0.0 rpy=0.0 0.0 0.0

Commit message: added ros_grbl

File: src/cnc_description/urdf/cnc.urdf (robot description, URDF)
Before this commit: robot cncweld, 5 links, 4 joints
Links:
- removed link X_axis
- removed link Y_axis
- removed link Z_axis
- added link X_link; collision mesh filename=package://cnc_description/meshes/X_axis.STL; visual mesh filename=package://cnc_description/meshes/X_axis.STL
- added link Y_link; collision mesh filename=package://cnc_description/meshes/Y_axis_assy.STL; visual mesh filename=package://cnc_description/meshes/Y_axis_assy.STL
- added link Z_link; collision mesh filename=package://cnc_description/meshes/Z_axis_assy.STL; visual mesh filename=package://cnc_description/meshes/Z_axis_assy.STL
Joints:
- removed joint X_axis_Y_axis_joint
- removed joint Y_axis_Z_axis_joint
- removed joint Z_axis_tool0_joint
- removed joint world_to_X_axis
- added joint X_link_Y_link_joint: type prismatic, parent X_link, child Y_link, origin xyz=0.0 0.0 0.0 rpy=0.0 0.0 0.0, axis 1 0 0, limit lower=0.0 upper=0.7 effort=1000.0 velocity=0.05
- added joint Y_link_Z_link_joint: type prismatic, parent Y_link, child Z_link, origin xyz=0.0 0.0 0.0 rpy=0.0 0.0 0.0, axis 0 1 0, limit lower=0.0 upper=0.21 effort=1000.0 velocity=0.05
- added joint Z_link_tool0_joint: type prismatic, parent Z_link, child tool0, origin xyz=0.31 0.046 0.0 rpy=0.0 0.0 0.0, axis 0 0 1, limit lower=0.0 upper=0.086 effort=1000.0 velocity=0.05
- added joint world_to_X_link: type fixed, parent world, child X_link, origin xyz=0.0 -0.1445 0.0 rpy=0.0 0.0 0.0

Commit message: moved onto desktop computer

File: src/cnc_description/urdf/cnc.urdf (robot description, URDF)
Before this commit: robot cncweld, 5 links, 4 joints
Links:
- removed link Y_link
- added link base_link; collision mesh filename=package://cnc_description/meshes/base_link.STL; visual mesh filename=package://cnc_description/meshes/base_link.STL
- link X_link: geometry collision mesh filename=package://cnc_description/meshes/X_link.STL; visual mesh filename=package://cnc_description/meshes/X_link.STL
Joints:
- removed joint X_link_Y_link_joint
- removed joint Y_link_Z_link_joint
- removed joint world_to_X_link
- added joint X_link_Z_link_joint: type prismatic, parent X_link, child Z_link, origin xyz=0.0 0.0 0.0 rpy=0.0 0.0 0.0, axis 0 1 0, limit lower=0.0 upper=0.21 effort=1000.0 velocity=0.05
- added joint base_link_X_link_joint: type prismatic, parent base_link, child X_link, origin xyz=0.05 0.0 0.083 rpy=0.0 0.0 0.0, axis 1 0 0, limit lower=0.0 upper=1.0 effort=1000.0 velocity=0.05
- added joint world_to_base_link: type fixed, parent world, child base_link, origin xyz=0.044 0.0 0.02 rpy=0.0 0.0 0.0

Commit message: 1st version of urdf with revolute joint A

File: src/cnc_description/urdf/cnc.urdf (robot description, URDF)
Before this commit: robot cncweld, 5 links, 4 joints
Links:
- removed link tool0
- added link Y_link; collision mesh filename=package://cnc_description/meshes/Y_link.STL; visual mesh filename=package://cnc_description/meshes/Y_link.STL
- added link torch; collision mesh filename=package://cnc_description/meshes/torch.STL; visual mesh filename=package://cnc_description/meshes/torch.STL
- added link torch_tip
- link Z_link: geometry collision mesh filename=package://cnc_description/meshes/Z_link.STL; visual mesh filename=package://cnc_description/meshes/Z_link.STL
Joints:
- removed joint X_link_Z_link_joint
- removed joint Z_link_tool0_joint
- added joint X_link_Y_link_joint: type prismatic, parent X_link, child Y_link, origin xyz=0.08 -0.058 -0.041 rpy=0.0 0.0 0.0, axis 0 1 0, limit lower=0.0 upper=0.18 effort=1000.0 velocity=0.05
- added joint Y_link_Z_link_joint: type prismatic, parent Y_link, child Z_link, origin xyz=0.068 0.0 0.23 rpy=0.0 0.0 0.0, axis 0 0 1, limit lower=-0.086 upper=0.0 effort=1000.0 velocity=0.05
- added joint Z_link_torch_joint: type revolute, parent Z_link, child torch, origin xyz=0.0 0.0 0.0 rpy=0.0 0.0 0.0, limit lower=-3.1416 upper=3.1416 effort=1000.0 velocity=0.05
- added joint torch_to_tip: type fixed, parent torch, child torch_tip, origin xyz=0.08 0.0 -0.19 rpy=0.0 0.0 0.0
- joint base_link_X_link_joint: limit lower=0.0 upper=1.0 effort=1000.0 velocity=0.05 -> lower=0.09 upper=0.75 effort=1000.0 velocity=0.05; origin xyz=0.05 0.0 0.083 rpy=0.0 0.0 0.0 -> xyz=0.0 0.0 0.083 rpy=0.0 0.0 0.0

Commit message: Added cncweld_support

File: src/cnc_description/urdf/cnc.urdf (robot description, URDF)
Before this commit: robot cncweld, 7 links, 6 joints
Links:
- removed link torch
- removed link torch_tip
- removed link world
- added link tool0
Joints:
- removed joint Z_link_torch_joint
- removed joint torch_to_tip
- removed joint world_to_base_link
- added joint Z_link_tool0: type revolute, parent Z_link, child tool0, origin xyz=0.0 0.0 0.0 rpy=0.0 0.0 0.0, limit lower=-3.1416 upper=3.1416 effort=1000.0 velocity=0.05

Commit message: development resume

File: src/cnc_description/urdf/cnc.urdf (robot description, URDF)
Before this commit: robot cncweld, 5 links, 4 joints
Links:
- added link sensor_optical_frame
- added link torch
- link tool0: geometry collision mesh filename=package://cnc_description/meshes/torch.STL; visual mesh filename=package://cnc_description/meshes/torch.STL
Joints:
- added joint tool0_sensor_optical_frame: type fixed, parent tool0, child sensor_optical_frame, origin xyz=0.082 0.0 -0.190 rpy=0.0 0.471238898038469 0.0
- added joint tool0_torch: type fixed, parent tool0, child torch, origin xyz=0.082 0.0 -0.190 rpy=0.0 0.0 0.0

Commit message: updated scanner optical from orientation

File: src/cnc_description/urdf/cnc.urdf (robot description, URDF)
Before this commit: robot cncweld, 7 links, 6 joints
Joints:
- joint X_link_Y_link_joint: origin xyz=0.08 -0.058 -0.041 rpy=0.0 0.0 0.0 -> xyz=0.08 -0.10 -0.041 rpy=0.0 0.0 0.0
- joint tool0_sensor_optical_frame: origin xyz=0.082 0.0 -0.190 rpy=0.0 0.471238898038469 0.0 -> xyz=0.082 0.0 -0.190 rpy=0.471238898038469 0.0 -1.5708

File: src/cncweld_support/urdf/cncweldKeyence.xacro (robot description, xacro)
@@ -63,5 +63,6 @@
   </link>
   <joint name="wrist_3_link-lj_v7200_fixed_joint" type="fixed">
-    <origin xyz="0.062 -0.105 0.1599" rpy="0 ${pi} ${-pi/2.0}"/>
+<!--    <origin xyz="0.062 -0.105 0.1599" rpy="0 ${pi} ${-pi/2.0}"/>-->
+    <origin xyz="0.062 -0.105 0.1599" rpy="0 ${pi} ${-pi}"/>
     <parent link="wrist_3_link"/>
     <child link="lj_v7200_frame"/>
