Commit message: cloned grbl_ros

File: src/cnc_description/urdf/cnc.xacro (robot description, xacro)
@@ -241,5 +241,5 @@
 -->
   <joint name="tool0_sensor_optical_frame" type="fixed">
-    <origin xyz="0.082 0.0 -0.190" rpy="0.471238898038469 0.0 -1.5708" />
+    <origin xyz="0.082 0.0 -0.190" rpy="0.471238898038469 0.0 ${-pi/2.0}" />
     <parent
       link="tool0" />

File: src/cncweld_support/urdf/cncweldKeyence.xacro (robot description, xacro)
@@ -4,23 +4,16 @@
 -->
 <robot xmlns:xacro="http://ros.org/wiki/xacro"
-       name="roboweld" >
-  <xacro:arg name="transmission_hw_interface" default="hardware_interface/PositionJointInterface"/>
-  <!-- ur5 -->
-  <xacro:include filename="$(find ur_description)/urdf/ur5.urdf.xacro" />
-  <!-- arm -->
-  <xacro:arg name="kinematics_config" default="$(find ur_description)/config/ur5_default.yaml"/>
-  <xacro:ur5_robot prefix="" joint_limited="true"
-    transmission_hw_interface="$(arg transmission_hw_interface)"
-    kinematics_file="${load_yaml('$(arg kinematics_config)')}"
-  />
-  <link name="world" />
+       name="cncweld" >
 <!-- There are:-
      1. The World, everything lives in it.
-     2. The Welding table, our robot arm is installed on it.
-     3. The Kinect V2, RGBD camera provides the point clouds that we need.
-     4. The UR5, our robot arm, with the Straight Fronius Torch as its end effector.
-     5. The Keyence LJ7200 Laser Scanner attached to the torch holder.
-     6. The RealSense D435i attached to the torch holder.
+     2. The cnc, the Self Built CNC Welding Mechanism with
+     3. The Straight Fronius Torch as its end effector together with its holder, and
+     4. The Keyence LJ7200 Laser Scanner attached to the torch holder.
 -->
+  <xacro:arg name="transmission_hw_interface" default="hardware_interface/PositionJointInterface"/>
+  <!-- The World that we are living in -->
+  <link name="world" />
+  <!-- The CNC machine -->
+  <xacro:include filename="$(find cnc_description)/urdf/cnc.urdf" />
   <!-- defining tool -->
   <!-- Welding torch holder with the Straight Torch -->

Commit message: Updated the scanner optical frame

File: src/cnc_description/urdf/cnc.xacro (robot description, xacro)
@@ -236,14 +236,14 @@
       link="torch" />
   </joint>
-<link name="sensor_optical_frame" />
+<link name="lj_v7200_optical_frame" />
 <!--
   The tool0 to keyence_optical_frame fixed Joint
 -->
-  <joint name="tool0_sensor_optical_frame" type="fixed">
+  <joint name="tool0_lj_v7200_optical_frame" type="fixed">
     <origin xyz="0.082 0.0 -0.190" rpy="0.471238898038469 0.0 ${-pi/2.0}" />
     <parent
       link="tool0" />
     <child
-      link="sensor_optical_frame" />
+      link="lj_v7200_optical_frame" />
   </joint>
 </robot>

Commit message: laser scanning added incomplete

File: src/cnc_description/urdf/cnc.xacro (robot description, xacro)
@@ -14,7 +14,15 @@
 -->
 <robot name="cncweld" xmlns:xacro="http://ros.org/wiki/xacro">
-<!--
   <link name="world" />
--->
+  <joint
+    name="world_base_link"
+    type="fixed">
+    <origin
+      xyz="0.0 0.0 0.0" rpy="0.0 0.0 0.0" />
+    <parent
+      link="world" />
+    <child
+      link="base_link" />
+  </joint>
 <!--
   There are 2 rails for the base link. The base_link.STL has already
@@ -237,4 +245,9 @@
   </joint>
 <link name="lj_v7200_optical_frame" />
+<joint name="optical_frame" type="fixed">
+  <origin xyz="0 0 0" rpy="0 0 0"/>
+  <parent link="lj_v7200_optical_frame"/>
+  <child link="lj_v7200_optical_frame"/>
+</joint>
 <!--
   The tool0 to keyence_optical_frame fixed Joint

Commit message: lj_v7200_optical_frame pose adjusted

File: src/cnc_description/urdf/cnc.xacro (robot description, xacro)
@@ -244,6 +244,6 @@
       link="torch" />
   </joint>
+<!--
 <link name="lj_v7200_optical_frame" />
-<!--
 <joint name="optical_frame" type="fixed">
   <origin xyz="0 0 0" rpy="0 0 0"/>
@@ -256,5 +256,5 @@
 -->
   <joint name="tool0_lj_v7200_optical_frame" type="fixed">
-    <origin xyz="0.082 0.0 -0.190" rpy="0.471238898038469 0.0 ${-pi/2.0}" />
+    <origin xyz="0.1083 0.000005 -0.19027" rpy="-0.471238898038469 0.0 ${-pi/2.0}" />
     <parent
       link="tool0" />
@@ -262,3 +262,5 @@
       link="lj_v7200_optical_frame" />
   </joint>
+  <xacro:include filename="$(find keyence_experimental)/urdf/lj_v7200_macro.xacro"/>
+  <xacro:lj_v7200 prefix=""/>
 </robot>

Commit message: waitForTransform problem resolved

File: src/cnc_description/urdf/cnc.xacro (robot description, xacro)
@@ -14,15 +14,4 @@
 -->
 <robot name="cncweld" xmlns:xacro="http://ros.org/wiki/xacro">
-  <link name="world" />
-  <joint
-    name="world_base_link"
-    type="fixed">
-    <origin
-      xyz="0.0 0.0 0.0" rpy="0.0 0.0 0.0" />
-    <parent
-      link="world" />
-    <child
-      link="base_link" />
-  </joint>
 <!--
   There are 2 rails for the base link. The base_link.STL has already

Commit message: base_link_X_link_joint changed height

File: src/cnc_description/urdf/cnc.xacro (robot description, xacro)
@@ -80,6 +80,9 @@
     name="base_link_X_link_joint"
     type="prismatic">
-    <origin
-      xyz="0.0 0.0 0.083" rpy="0.0 0.0 0.0" />
+<!--
+    <origin
+      xyz="0.0 0.0 0.083" rpy="0.0 0.0 0.0" /> -->
+    <origin
+      xyz="0.0 0.0 0.0998" rpy="0.0 0.0 0.0" />
     <parent
       link="base_link" />

Commit message: Optical frame pose adjusted

File: src/cnc_description/urdf/cnc.xacro (robot description, xacro)
@@ -12,6 +12,20 @@
                          is called the torch.
 Updated on 6 May 2022,   The Origin of the sensor_optical_frame was adjusted.
+updated on 26 May 2022,  A world link is added and a world to base_link fixed joint
+                         added. The is necessary for the base_link is above the bottom
+                         of the Device and fixed joint added is to lift the whole
+                         thing up by 16.8mm.
 -->
 <robot name="cncweld" xmlns:xacro="http://ros.org/wiki/xacro">
+<link name="world" />
+<!--
+  The world to base link fixed Joint
+-->
+  <joint name="world_base_link" type="fixed">
+<!--    <origin xyz="0.0 0.0 0.0168" rpy="0.0 0.0 0.0" /> -->
+    <origin xyz="0.0 0.0 0.02" rpy="0.0 0.0 0.0" />
+    <parent link="world" />
+    <child  link="base_link" />
+  </joint>
 <!--
   There are 2 rails for the base link. The base_link.STL has already
@@ -80,9 +94,9 @@
     name="base_link_X_link_joint"
     type="prismatic">
-<!--
     <origin
-      xyz="0.0 0.0 0.083" rpy="0.0 0.0 0.0" /> -->
+      xyz="0.0 0.0 0.083" rpy="0.0 0.0 0.0" />
+<!--
     <origin
-      xyz="0.0 0.0 0.0998" rpy="0.0 0.0 0.0" />
+      xyz="0.0 0.0 0.0998" rpy="0.0 0.0 0.0" /> -->
     <parent
       link="base_link" />
@@ -131,6 +145,6 @@
       xyz="0.08 -0.058 -0.041" rpy="0.0 0.0 0.0" />
     -->
-    <origin
-      xyz="0.08 -0.10 -0.041" rpy="0.0 0.0 0.0" />
+<!--    <origin xyz="0.08 -0.10 -0.041" rpy="0.0 0.0 0.0" /> -->
+    <origin xyz="0.08 -0.10 -0.05" rpy="0.0 0.0 0.0" />
     <parent
       link="X_link" />
@@ -248,5 +262,8 @@
 -->
   <joint name="tool0_lj_v7200_optical_frame" type="fixed">
+<!--
     <origin xyz="0.1083 0.000005 -0.19027" rpy="-0.471238898038469 0.0 ${-pi/2.0}" />
+-->
+    <origin xyz="0.1083 0.000005 -0.18527" rpy="-0.471238898038469 0.0 ${-pi/2.0}" />
     <parent
       link="tool0" />
