Commit message: 2nd commit

File: src/cncweld_description/urdf/O-cncweld.xacro (robot description, xacro)
@@ -17,6 +17,4 @@
                          thing up by 16.8mm.
 Updated on 23 June, 2022.World is moved to direcly under torch.
-11 October 2022. for the 3rd branch.
-This is new for the Consealed Lead Screws.
 -->
 <robot name="robot_description" xmlns:xacro="http://ros.org/wiki/xacro">
@@ -254,4 +252,12 @@
   </joint>
 <!--
+<link name="lj_v7200_optical_frame" />
+<joint name="optical_frame" type="fixed">
+  <origin xyz="0 0 0" rpy="0 0 0"/>
+  <parent link="lj_v7200_optical_frame"/>
+  <child link="lj_v7200_optical_frame"/>
+</joint>
+-->
+<!--
   The tool0 to keyence_optical_frame fixed Joint
 -->
