Commit message: core using libserial, devel jsp

File: src/cncweld_description/urdf/cncweld.xacro (robot description, xacro)
@@ -17,5 +17,5 @@
                          thing up by 16.8mm.
 -->
-<robot name="cncweld" xmlns:xacro="http://ros.org/wiki/xacro">
+<robot name="robot_description" xmlns:xacro="http://ros.org/wiki/xacro">
 <link name="world" />
 <!--
@@ -40,5 +40,5 @@
       <geometry>
         <mesh
-          filename="package://cnc_description/meshes/base_link.STL" />
+          filename="package://cncweld_description/meshes/base_link.STL" />
       </geometry>
       <material
@@ -54,5 +54,5 @@
       <geometry>
         <mesh
-          filename="package://cnc_description/meshes/base_link.STL" />
+          filename="package://cncweld_description/meshes/base_link.STL" />
       </geometry>
     </collision>
@@ -70,19 +70,19 @@
       <geometry>
         <mesh
-          filename="package://cnc_description/meshes/X_link.STL" />
-      </geometry>
-      <material
-        name="">
-        <color
-          rgba="0.792156862745098 0.819607843137255 0.933333333333333 1" />
-      </material>
-    </visual>
-    <collision>
-      <origin
-        xyz="0.0 0.0 0.0"
-        rpy="0 0 0" />
-      <geometry>
-        <mesh
-          filename="package://cnc_description/meshes/X_link.STL" />
+          filename="package://cncweld_description/meshes/X_link.STL" />
+      </geometry>
+      <material
+        name="">
+        <color
+          rgba="0.792156862745098 0.819607843137255 0.933333333333333 1" />
+      </material>
+    </visual>
+    <collision>
+      <origin
+        xyz="0.0 0.0 0.0"
+        rpy="0 0 0" />
+      <geometry>
+        <mesh
+          filename="package://cncweld_description/meshes/X_link.STL" />
       </geometry>
     </collision>
@@ -117,19 +117,19 @@
       <geometry>
         <mesh
-          filename="package://cnc_description/meshes/Y_link.STL" />
-      </geometry>
-      <material
-        name="">
-        <color
-          rgba="0.792156862745098 0.819607843137255 0.933333333333333 1" />
-      </material>
-    </visual>
-    <collision>
-      <origin
-        xyz="0.0 0.0 0.0"
-        rpy="0 0 0" />
-      <geometry>
-        <mesh
-          filename="package://cnc_description/meshes/Y_link.STL" />
+          filename="package://cncweld_description/meshes/Y_link.STL" />
+      </geometry>
+      <material
+        name="">
+        <color
+          rgba="0.792156862745098 0.819607843137255 0.933333333333333 1" />
+      </material>
+    </visual>
+    <collision>
+      <origin
+        xyz="0.0 0.0 0.0"
+        rpy="0 0 0" />
+      <geometry>
+        <mesh
+          filename="package://cncweld_description/meshes/Y_link.STL" />
       </geometry>
     </collision>
@@ -165,19 +165,19 @@
       <geometry>
         <mesh
-          filename="package://cnc_description/meshes/Z_link.STL" />
-      </geometry>
-      <material
-        name="">
-        <color
-          rgba="0.792156862745098 0.819607843137255 0.933333333333333 1" />
-      </material>
-    </visual>
-    <collision>
-      <origin
-        xyz="0.0 0.0 0.0"
-        rpy="0 0 0" />
-      <geometry>
-        <mesh
-          filename="package://cnc_description/meshes/Z_link.STL" />
+          filename="package://cncweld_description/meshes/Z_link.STL" />
+      </geometry>
+      <material
+        name="">
+        <color
+          rgba="0.792156862745098 0.819607843137255 0.933333333333333 1" />
+      </material>
+    </visual>
+    <collision>
+      <origin
+        xyz="0.0 0.0 0.0"
+        rpy="0 0 0" />
+      <geometry>
+        <mesh
+          filename="package://cncweld_description/meshes/Z_link.STL" />
       </geometry>
     </collision>
@@ -221,19 +221,19 @@
       <geometry>
         <mesh
-          filename="package://cnc_description/meshes/torch.STL" />
-      </geometry>
-      <material
-        name="">
-        <color
-          rgba="0.792156862745098 0.819607843137255 0.933333333333333 1" />
-      </material>
-    </visual>
-    <collision>
-      <origin
-        xyz="0.0 0.0 0.0"
-        rpy="0 0 0" />
-      <geometry>
-        <mesh
-          filename="package://cnc_description/meshes/torch.STL" />
+          filename="package://cncweld_description/meshes/torch.STL" />
+      </geometry>
+      <material
+        name="">
+        <color
+          rgba="0.792156862745098 0.819607843137255 0.933333333333333 1" />
+      </material>
+    </visual>
+    <collision>
+      <origin
+        xyz="0.0 0.0 0.0"
+        rpy="0 0 0" />
+      <geometry>
+        <mesh
+          filename="package://cncweld_description/meshes/torch.STL" />
       </geometry>
     </collision>

Commit message: kind of working but not quite yet

File: src/cncweld_description/urdf/cncweld.xacro (robot description, xacro)
@@ -95,5 +95,5 @@
     type="prismatic">
     <origin
-      xyz="0.0 0.0 0.083" rpy="0.0 0.0 0.0" />
+      xyz="0.09 0.0 0.083" rpy="0.0 0.0 0.0" />
 <!--
     <origin
@@ -146,5 +146,5 @@
     -->
 <!--    <origin xyz="0.08 -0.10 -0.041" rpy="0.0 0.0 0.0" /> -->
-    <origin xyz="0.08 -0.10 -0.05" rpy="0.0 0.0 0.0" />
+    <origin xyz="0.08 -0.09 -0.05" rpy="0.0 0.0 0.0" />
     <parent
       link="X_link" />

Commit message: the world (frame) moved

File: src/cncweld_description/urdf/cncweld.xacro (robot description, xacro)
@@ -16,4 +16,5 @@
                          of the Device and fixed joint added is to lift the whole
                          thing up by 16.8mm.
+Updated on 23 June, 2022.World is moved to direcly under torch.
 -->
 <robot name="robot_description" xmlns:xacro="http://ros.org/wiki/xacro">
@@ -24,5 +25,5 @@
   <joint name="world_base_link" type="fixed">
 <!--    <origin xyz="0.0 0.0 0.0168" rpy="0.0 0.0 0.0" /> -->
-    <origin xyz="0.0 0.0 0.02" rpy="0.0 0.0 0.0" />
+    <origin xyz="-0.32 0.09 0.02" rpy="0.0 0.0 0.0" />
     <parent link="world" />
     <child  link="base_link" />
@@ -95,5 +96,5 @@
     type="prismatic">
     <origin
-      xyz="0.09 0.0 0.083" rpy="0.0 0.0 0.0" />
+      xyz="0.09 0.00 0.083" rpy="0.0 0.0 0.0" />
 <!--
     <origin
@@ -104,5 +105,5 @@
       link="X_link" />
     <axis  xyz="1 0 0"/>
-    <limit effort="1000.0" lower="0.09" upper="0.75" velocity="0.05"/>
+    <limit effort="100.0" lower="0.0" upper="0.75" velocity="0.05"/>
   </joint>
 <!--
@@ -151,5 +152,5 @@
     <child
       link="Y_link" />
-    <limit effort="1000.0" lower="0.0" upper="0.18" velocity="0.05"/>
+    <limit effort="1000.0" lower="-0.5" upper="0.2" velocity="0.05"/>
     <axis  xyz="0 1 0"/>
   </joint>

Commit message: curvy path

File: src/cncweld_description/urdf/cncweld.xacro (robot description, xacro)
@@ -152,5 +152,5 @@
     <child
       link="Y_link" />
-    <limit effort="1000.0" lower="-0.5" upper="0.2" velocity="0.05"/>
+    <limit effort="100.0" lower="0.0" upper="0.2" velocity="0.05"/>
     <axis  xyz="0 1 0"/>
   </joint>
@@ -198,5 +198,5 @@
     <child
       link="Z_link" />
-    <limit effort="1000.0" lower="-0.086" upper="0.0" velocity="0.05"/>
+    <limit effort="100.0" lower="-0.086" upper="0.0" velocity="0.05"/>
     <axis  xyz="0 0 1"/>
   </joint>
@@ -210,5 +210,5 @@
     <child
       link="tool0" />
-    <limit effort="1000.0" lower="-3.1416" upper="3.1416" velocity="0.05"/>
+    <limit effort="100.0" lower="-3.1416" upper="3.1416" velocity="0.05"/>
   </joint>
 <!--

Commit message: again

File: src/cncweld_description/urdf/cncweld.xacro (robot description, xacro)
@@ -186,85 +186,3 @@
     </collision>
   </link>
-<!--
-  The Y link to Z_link Prismatic Joint
--->
-  <joint
-    name="Y_link_Z_link_joint"
-    type="prismatic">
-<!--
-    <origin xyz="0.045 0.0 0.0" rpy="0.0 0.0 0.0" />
--->
-    <origin xyz="0.068 0.0 0.23" rpy="0.0 0.0 0.0" />
-    <parent
-      link="Y_link" />
-    <child
-      link="Z_link" />
-    <limit effort="100.0" lower="-0.086" upper="0.0" velocity="0.05"/>
-    <axis  xyz="0 0 1"/>
-  </joint>
-<!--
-  The Z_link to tool0 Revolute Joint
--->
-  <joint name="Z_link_tool0" type="revolute">
-    <origin xyz="0.0 0.0 0.0" rpy="0.0 0.0 0.0" />
-    <parent
-      link="Z_link" />
-    <child
-      link="tool0" />
-    <limit effort="100.0" lower="-3.1416" upper="3.1416" velocity="0.05"/>
-  </joint>
-<!--
-  The tool0 link
--->
-  <link name="tool0">
-    <visual>
-      <origin
-        xyz="0.0 0.0 0.0"
-        rpy="0 0 0" />
-      <geometry>
-        <mesh
-          filename="package://cncweld_description/meshes/torch.STL" />
-      </geometry>
-      <material
-        name="">
-        <color
-          rgba="0.792156862745098 0.819607843137255 0.933333333333333 1" />
-      </material>
-    </visual>
-    <collision>
-      <origin
-        xyz="0.0 0.0 0.0"
-        rpy="0 0 0" />
-      <geometry>
-        <mesh
-          filename="package://cncweld_description/meshes/torch.STL" />
-      </geometry>
-    </collision>
-  </link>
-<link name="torch" />
-<!--
-  The tool0 to torch fixed Joint
--->
-  <joint name="tool0_torch" type="fixed">
-    <origin xyz="0.082 0.0 -0.190" rpy="0.0 0.0 0.0" />
-    <parent
-      link="tool0" />
-    <child
-      link="torch" />
-  </joint>
-<!--
-  The tool0 to keyence_optical_frame fixed Joint
--->
-  <joint name="tool0_lj_v7200_optical_frame" type="fixed">
-<!--
-    <origin xyz="0.1083 0.000005 -0.19027" rpy="-0.471238898038469 0.0 ${-pi/2.0}" />
--->
-    <origin xyz="0.1083 0.000005 -0.18527" rpy="-0.471238898038469 0.0 ${-pi/2.0}" />
-    <parent
-      link="tool0" />
-    <child
-      link="lj_v7200_optical_frame" />
-  </joint>
-  <xacro:include filename="$(find keyence_experimental)/urdf/lj_v7200_macro.xacro"/>
-  <xacro:lj_v7200 prefix=""/>
 </robot>

Commit message: Still testing

File: src/cncweld_description/urdf/cncweld.xacro (robot description, xacro)
@@ -26,6 +26,5 @@
 -->
   <joint name="world_base_link" type="fixed">
-<!--    <origin xyz="0.0 0.0 0.0168" rpy="0.0 0.0 0.0" /> -->
-    <origin xyz="-0.32 0.09 0.02" rpy="0.0 0.0 0.0" />
+    <origin xyz="0 0 0" rpy="0.0 0.0 0.0" />
     <parent link="world" />
     <child  link="base_link" />
@@ -144,9 +143,4 @@
     name="X_link_Y_link_joint"
     type="prismatic">
-    <!--
-    <origin
-      xyz="0.08 -0.058 -0.041" rpy="0.0 0.0 0.0" />
-    -->
-<!--    <origin xyz="0.08 -0.10 -0.041" rpy="0.0 0.0 0.0" /> -->
     <origin xyz="0.08 -0.09 -0.05" rpy="0.0 0.0 0.0" />
     <parent
@@ -186,3 +180,20 @@
     </collision>
   </link>
+<!--
+  The Y link to Z_link Prismatic Joint
+-->
+  <joint
+    name="Y_link_Z_link_joint"
+    type="prismatic">
+<!--
+    <origin xyz="0.045 0.0 0.0" rpy="0.0 0.0 0.0" />
+-->
+    <origin xyz="0.068 0.0 0.23" rpy="0.0 0.0 0.0" />
+    <parent
+      link="Y_link" />
+    <child
+      link="Z_link" />
+    <limit effort="100.0" lower="-0.086" upper="0.0" velocity="0.05"/>
+    <axis  xyz="0 0 1"/>
+  </joint>
 </robot>

Commit message: Still working on the urdf

File: src/cncweld_description/urdf/cncweld.xacro (robot description, xacro)
@@ -97,8 +97,5 @@
     type="prismatic">
     <origin
-      xyz="0.09 0.00 0.083" rpy="0.0 0.0 0.0" />
-<!--
-    <origin
-      xyz="0.0 0.0 0.0998" rpy="0.0 0.0 0.0" /> -->
+      xyz="0.0 0.00 0.0" rpy="0.0 0.0 0.0" />
     <parent
       link="base_link" />
@@ -143,5 +140,5 @@
     name="X_link_Y_link_joint"
     type="prismatic">
-    <origin xyz="0.08 -0.09 -0.05" rpy="0.0 0.0 0.0" />
+    <origin xyz="0.0 -0.0 -0.0" rpy="0.0 0.0 0.0" />
     <parent
       link="X_link" />
@@ -186,8 +183,5 @@
     name="Y_link_Z_link_joint"
     type="prismatic">
-<!--
-    <origin xyz="0.045 0.0 0.0" rpy="0.0 0.0 0.0" />
--->
-    <origin xyz="0.068 0.0 0.23" rpy="0.0 0.0 0.0" />
+    <origin xyz="0.0 0.0 0.0" rpy="0.0 0.0 0.0" />
     <parent
       link="Y_link" />

Commit message: origins done to base link, x link and z link

File: src/cncweld_description/urdf/cncweld.xacro (robot description, xacro)
@@ -26,5 +26,5 @@
 -->
   <joint name="world_base_link" type="fixed">
-    <origin xyz="0 0 0" rpy="0.0 0.0 0.0" />
+    <origin xyz="0 -0.25 0" rpy="0.0 0.0 0.0" />
     <parent link="world" />
     <child  link="base_link" />
@@ -97,5 +97,5 @@
     type="prismatic">
     <origin
-      xyz="0.0 0.00 0.0" rpy="0.0 0.0 0.0" />
+      xyz="0.11 0.00 0.1" rpy="0.0 0.0 0.0" />
     <parent
       link="base_link" />

Commit message: cncweld.xacro debugged

File: src/cncweld_description/urdf/cncweld.xacro (robot description, xacro)
@@ -140,10 +140,10 @@
     name="X_link_Y_link_joint"
     type="prismatic">
-    <origin xyz="0.0 -0.0 -0.0" rpy="0.0 0.0 0.0" />
+    <origin xyz="0.095 0.064 -0.041" rpy="0.0 0.0 0.0" />
     <parent
       link="X_link" />
     <child
       link="Y_link" />
-    <limit effort="100.0" lower="0.0" upper="0.2" velocity="0.05"/>
+    <limit effort="100.0" lower="0.0" upper="0.365" velocity="0.05"/>
     <axis  xyz="0 1 0"/>
   </joint>
@@ -183,10 +183,10 @@
     name="Y_link_Z_link_joint"
     type="prismatic">
-    <origin xyz="0.0 0.0 0.0" rpy="0.0 0.0 0.0" />
+    <origin xyz="0.016 0.0 0.2855" rpy="0.0 0.0 0.0" />
     <parent
       link="Y_link" />
     <child
       link="Z_link" />
-    <limit effort="100.0" lower="-0.086" upper="0.0" velocity="0.05"/>
+    <limit effort="100.0" lower="-0.221" upper="0.0" velocity="0.05"/>
     <axis  xyz="0 0 1"/>
   </joint>

Commit message: setuptest.launch works

File: src/cncweld_description/urdf/cncweld.xacro (robot description, xacro)
@@ -191,3 +191,43 @@
     <axis  xyz="0 0 1"/>
   </joint>
+<!--
+  The torch on the torch holder
+-->
+  <link name="torch" >
+    <visual>
+      <origin
+        xyz="0.0 0.0 0.0"
+        rpy="0 0 0" />
+      <geometry>
+        <mesh
+          filename="package://cncweld_support/meshes/mere_torch.STL"
+          scale="0.001 0.001 0.001" />
+      </geometry>
+      <material
+        name="">
+        <color
+          rgba="0.792156862745098 0.819607843137255 0.933333333333333 1" />
+      </material>
+    </visual>
+    <collision>
+      <origin
+        xyz="0.0 0.0 0.0"
+        rpy="0 0 0" />
+      <geometry>
+        <mesh
+          filename="package://cncweld_support/meshes/mere_torch.STL"
+          scale="0.001 0.001 0.001" />
+      </geometry>
+    </collision>
+  </link>
+<!--
+  Z_link to torch fixed Joint
+-->
+  <joint name="Z_link_torch" type="fixed">
+    <origin xyz="0.0 0.0 0.0" rpy="0.0 0.0 0.0" />
+    <parent
+      link="Z_link" />
+    <child
+      link="torch" />
+  </joint>
 </robot>

Commit message: camera sorted out as well in rviz

File: src/cncweld_description/urdf/cncweld.xacro (robot description, xacro)
@@ -231,3 +231,20 @@
       link="torch" />
   </joint>
+<!--
+  Torch to Torch tip
+-->
+  <link name="TorchTip" />
+  <joint name="Torch_to_TorchTip" type="fixed">
+    <origin xyz="0.08 0.0 -0.215" rpy="0.0 0.0 0.0" />
+    <parent link="torch" />
+    <child  link="TorchTip" />
+  </joint>
+<!--
+  The Intel RealSense RGBD camera D435i
+-->
+  <!-- Import the realsense D435i description -->
+  <xacro:include filename="$(find realsense2_description)/urdf/_d435.urdf.xacro" />
+  <xacro:sensor_d435 parent="Z_link" use_nominal_extrinsics="true" name="d435i">
+    <origin xyz=" 0.14515 0 -0.025" rpy="${pi} ${pi/2} ${pi}"/>
+  </xacro:sensor_d435>
 </robot>

Commit message: Adding bottom

File: src/cncweld_description/urdf/cncweld.xacro (robot description, xacro)
@@ -22,6 +22,34 @@
 <robot name="robot_description" xmlns:xacro="http://ros.org/wiki/xacro">
 <link name="world" />
-<!--
-  The world to base link fixed Joint
+  <link name="bottom" >
+    <visual>
+      <origin
+        xyz="0 0 0"
+        rpy="0 0 0" />
+      <geometry>
+        <mesh
+          filename="package://cncweld_support/meshes/bottom.STL" />
+      </geometry>
+      <material
+        name="">
+        <color
+          rgba="0.792156862745098 0.819607843137255 0.933333333333333 1" />
+      </material>
+    </visual>
+    <collision>
+      <origin
+        xyz="0 0 0"
+        rpy="0 0 0" />
+      <geometry>
+        <mesh
+          filename="package://cncweld_support/meshes/bottom.STL" />
+      </geometry>
+    </collision>
+  </link>
+<!--
+  The world to bottom link fixed Joint
+-->
+<!--
+  The bottom to base link fixed Joint
 -->
   <joint name="world_base_link" type="fixed">

Commit message: Bottom fixed

File: src/cncweld_description/urdf/cncweld.xacro (robot description, xacro)
@@ -22,38 +22,80 @@
 <robot name="robot_description" xmlns:xacro="http://ros.org/wiki/xacro">
 <link name="world" />
-  <link name="bottom" >
-    <visual>
-      <origin
-        xyz="0 0 0"
-        rpy="0 0 0" />
-      <geometry>
-        <mesh
-          filename="package://cncweld_support/meshes/bottom.STL" />
-      </geometry>
-      <material
-        name="">
-        <color
-          rgba="0.792156862745098 0.819607843137255 0.933333333333333 1" />
-      </material>
-    </visual>
-    <collision>
-      <origin
-        xyz="0 0 0"
-        rpy="0 0 0" />
-      <geometry>
-        <mesh
-          filename="package://cncweld_support/meshes/bottom.STL" />
-      </geometry>
-    </collision>
-  </link>
+<link name="bottom" >
+  <visual>
+    <origin
+      xyz="0 0 0"
+      rpy="0 0 0" />
+    <geometry>
+      <mesh
+        filename="package://cncweld_support/meshes/bottom.STL"
+        scale="0.001 0.001 0.001" />
+    </geometry>
+    <material
+      name="">
+      <color
+        rgba="0.792156862745098 0.819607843137255 0.933333333333333 1" />
+    </material>
+  </visual>
+  <collision>
+    <origin
+      xyz="0 0 0"
+      rpy="0 0 0" />
+    <geometry>
+      <mesh
+        filename="package://cncweld_support/meshes/bottom.STL"
+        scale="0.001 0.001 0.001" />
+    </geometry>
+  </collision>
+</link>
+<link name="bottom2" >
+  <visual>
+    <origin
+      xyz="0 0 0"
+      rpy="0 0 0" />
+    <geometry>
+      <mesh
+        filename="package://cncweld_support/meshes/bottom.STL"
+        scale="0.001 0.001 0.001" />
+    </geometry>
+    <material
+      name="">
+      <color
+        rgba="0.792156862745098 0.819607843137255 0.933333333333333 1" />
+    </material>
+  </visual>
+  <collision>
+    <origin
+      xyz="0 0 0"
+      rpy="0 0 0" />
+    <geometry>
+      <mesh
+        filename="package://cncweld_support/meshes/bottom.STL"
+        scale="0.001 0.001 0.001" />
+    </geometry>
+  </collision>
+</link>
 <!--
   The world to bottom link fixed Joint
 -->
+  <joint name="world_bottom" type="fixed">
+    <origin xyz="1.177 0.280 0.025" rpy="0.0 0.0 0.0" />
+    <parent link="world" />
+    <child  link="bottom" />
+  </joint>
+<!--
+  The world to bottom2 link fixed Joint
+-->
+  <joint name="world_bottom2" type="fixed">
+    <origin xyz="1.177 -0.280 0.025" rpy="0.0 0.0 0.0" />
+    <parent link="world" />
+    <child  link="bottom2" />
+  </joint>
 <!--
   The bottom to base link fixed Joint
 -->
-  <joint name="world_base_link" type="fixed">
-    <origin xyz="0 -0.25 0" rpy="0.0 0.0 0.0" />
-    <parent link="world" />
+  <joint name="bottom_base_link" type="fixed">
+    <origin xyz="-1.177 -0.530 0.025" rpy="0.0 0.0 0.0" />
+    <parent link="bottom" />
     <child  link="base_link" />
   </joint>

Commit message: Back to Keyence

File: src/cncweld_description/urdf/cncweld.xacro (robot description, xacro)
@@ -19,4 +19,5 @@
 11 October 2022. for the 3rd branch.
 This is new for the Consealed Lead Screws.
+25 November 2022. for Demonstration with the Keyence scanner.
 -->
 <robot name="robot_description" xmlns:xacro="http://ros.org/wiki/xacro">
@@ -313,8 +314,32 @@
   The Intel RealSense RGBD camera D435i
 -->
-  <!-- Import the realsense D435i description -->
+  <!-- Import the realsense D435i description
   <xacro:include filename="$(find realsense2_description)/urdf/_d435.urdf.xacro" />
   <xacro:sensor_d435 parent="Z_link" use_nominal_extrinsics="true" name="d435i">
     <origin xyz=" 0.14515 0 -0.025" rpy="${pi} ${pi/2} ${pi}"/>
   </xacro:sensor_d435>
+-->
+<!--
+<link name="lj_v7200_optical_frame" />
+<joint name="optical_frame" type="fixed">
+  <origin xyz="0 0 0" rpy="0 0 0"/>
+  <parent link="lj_v7200_optical_frame"/>
+  <child link="lj_v7200_optical_frame"/>
+</joint>
+-->
+<!--
+  The Z_link to keyence_optical_frame fixed Joint
+-->
+  <joint name="Z_link_lj_v7200_optical_frame" type="fixed">
+<!--
+    <origin xyz="0.1083 0.000005 -0.19027" rpy="-0.471238898038469 0.0 ${-pi/2.0}" />
+-->
+    <origin xyz="0.1083 0.000005 -0.18527" rpy="-0.471238898038469 0.0 ${-pi/2.0}" />
+    <parent
+      link="Z_link" />
+    <child
+      link="lj_v7200_optical_frame" />
+  </joint>
+  <xacro:include filename="$(find keyence_experimental)/urdf/lj_v7200_macro.xacro"/>
+  <xacro:lj_v7200 prefix=""/>
 </robot>

Commit message: All position correctly

File: src/cncweld_description/urdf/cncweld.xacro (robot description, xacro)
@@ -211,5 +211,8 @@
     name="X_link_Y_link_joint"
     type="prismatic">
+<!--
     <origin xyz="0.095 0.064 -0.041" rpy="0.0 0.0 0.0" />
+-->
+    <origin xyz="0.095 0.064 -0.031" rpy="0.0 0.0 0.0" />
     <parent
       link="X_link" />
@@ -264,5 +267,4 @@
 <!--
   The torch on the torch holder
--->
   <link name="torch" >
     <visual>
@@ -288,4 +290,32 @@
         <mesh
           filename="package://cncweld_support/meshes/mere_torch.STL"
+          scale="0.001 0.001 0.001" />
+      </geometry>
+    </collision>
+  </link>
+-->
+  <link name="torch" >
+    <visual>
+      <origin
+        xyz="0.0 0.0 0.0"
+        rpy="0 0 0" />
+      <geometry>
+        <mesh
+          filename="package://cncweld_support/meshes/scanner_holder.stl"
+          scale="0.001 0.001 0.001" />
+      </geometry>
+      <material
+        name="">
+        <color
+          rgba="0.792156862745098 0.819607843137255 0.933333333333333 1" />
+      </material>
+    </visual>
+    <collision>
+      <origin
+        xyz="0.0 0.0 0.0"
+        rpy="0 0 0" />
+      <geometry>
+        <mesh
+          filename="package://cncweld_support/meshes/scanner_holder.stl"
           scale="0.001 0.001 0.001" />
       </geometry>
@@ -335,5 +365,5 @@
     <origin xyz="0.1083 0.000005 -0.19027" rpy="-0.471238898038469 0.0 ${-pi/2.0}" />
 -->
-    <origin xyz="0.1083 0.000005 -0.18527" rpy="-0.471238898038469 0.0 ${-pi/2.0}" />
+    <origin xyz="0.10812 0.003 -0.21544" rpy="-0.471238898038469 0.0 ${-pi/2.0}" />
     <parent
       link="Z_link" />
